File: MinipHV2_1.brd (EAGLE design)
At the start: 27.9 x 27.9 mm, 33 parts, among them IC1 MCP3221, IC4 TL072, IC5 TPS60400DBV

Commit message: updated design files to v2_1
Parts:
- moved C9 3.05 mm to (15.5, 14.2)
- moved R8 1.52 mm to (15.5, 12.7)
- moved R7 1.52 mm to (15.5, 11.2)
Routing:
- net N$10: track 26.7 -> 17.2 mm, vias 2 -> 0
Changed lines of the file:
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@@
 <text x="23.876" y="7.112" size="0.6096" layer="21">Ver 0.1</text>
 <rectangle x1="17.78" y1="5.842" x2="27.178" y2="8.89" layer="22" rot="R180"/>
+<rectangle x1="14.986" y1="5.842" x2="17.78" y2="8.89" layer="22"/>
 </plain>
 <attributes>
@@
 <element name="IC4" library="SparkysWidgets" package="SO08" value="TL072" x="12.192" y="19.558" smashed="yes" rot="MR0"/>
 <element name="IC5" library="SparkysWidgets" package="SOT23-DBV" value="TPS60400DBV" x="4.318" y="14.732" smashed="yes" rot="MR270"/>
-<element name="R7" library="SparkysWidgets" package="0805" value="47K" x="15.494" y="12.7" smashed="yes" rot="MR0">
-<attribute name="NAME" x="18.542" y="13.0175" size="0.4064" layer="26" rot="MR0"/>
-<attribute name="VALUE" x="18.542" y="12.319" size="0.4064" layer="28" rot="MR0"/>
-</element>
-<element name="R8" library="SparkysWidgets" package="0805" value="220K" x="15.494" y="14.224" smashed="yes" rot="MR180">
-<attribute name="NAME" x="18.796" y="14.7955" size="0.4064" layer="26" rot="MR0"/>
-<attribute name="VALUE" x="18.796" y="14.097" size="0.4064" layer="28" rot="MR0"/>
+<element name="R7" library="SparkysWidgets" package="0805" value="47K" x="15.494" y="11.176" smashed="yes" rot="MR0">
+<attribute name="NAME" x="18.542" y="11.4935" size="0.4064" layer="26" rot="MR0"/>
+<attribute name="VALUE" x="18.542" y="10.795" size="0.4064" layer="28" rot="MR0"/>
+</element>
+<element name="R8" library="SparkysWidgets" package="0805" value="220K" x="15.494" y="12.7" smashed="yes" rot="MR180">
+<attribute name="NAME" x="18.796" y="13.2715" size="0.4064" layer="26" rot="MR0"/>
+<attribute name="VALUE" x="18.796" y="12.573" size="0.4064" layer="28" rot="MR0"/>
 </element>
 <element name="R9" library="SparkysWidgets" package="0805" value="220K" x="8.382" y="24.384" smashed="yes" rot="MR90">
@@
 <attribute name="VALUE" x="15.494" y="23.495" size="0.4064" layer="27"/>
 </element>
-<element name="C9" library="SparkysWidgets" package="0805" value=".1uF" x="15.494" y="11.176" smashed="yes" rot="MR0">
-<attribute name="NAME" x="18.542" y="11.2395" size="0.4064" layer="26" rot="MR0"/>
-<attribute name="VALUE" x="18.542" y="10.541" size="0.4064" layer="28" rot="MR0"/>
+<element name="C9" library="SparkysWidgets" package="0805" value=".1uF" x="15.494" y="14.224" smashed="yes" rot="MR0">
+<attribute name="NAME" x="18.542" y="14.2875" size="0.4064" layer="26" rot="MR0"/>
+<attribute name="VALUE" x="18.542" y="13.589" size="0.4064" layer="28" rot="MR0"/>
 </element>
 <element name="R12" library="SparkysWidgets" package="0805" value="3K" x="10.414" y="25.4" smashed="yes" rot="R270">
@@
 <wire x1="11.176" y1="18.542" x2="13.208" y2="18.542" width="0.254" layer="16"/>
 <wire x1="13.208" y1="18.542" x2="13.462" y2="18.288" width="0.254" layer="16"/>
-<wire x1="13.716" y1="14.224" x2="14.594" y2="14.224" width="0.254" layer="16"/>
+<wire x1="14.594" y1="11.176" x2="14.594" y2="12.7" width="0.254" layer="16"/>
 <wire x1="14.594" y1="12.7" x2="14.594" y2="14.224" width="0.254" layer="16"/>
-<wire x1="14.594" y1="11.176" x2="14.594" y2="12.7" width="0.254" layer="16"/>
+<wire x1="14.594" y1="14.224" x2="13.716" y2="14.224" width="0.254" layer="16"/>
 <wire x1="14.594" y1="14.224" x2="15.494" y2="14.224" width="0.254" layer="16"/>
 </signal>
@@
 <contactref element="R9" pad="1"/>
 <contactref element="R8" pad="2"/>
-<wire x1="16.394" y1="11.176" x2="16.394" y2="9.536" width="0.254" layer="16"/>
-<wire x1="16.394" y1="9.536" x2="15.494" y2="8.636" width="0.254" layer="16"/>
-<via x="15.494" y="8.636" extent="1-16" drill="0.6"/>
-<wire x1="15.494" y1="8.636" x2="15.494" y2="16.51" width="0.254" layer="1"/>
-<via x="15.494" y="16.51" extent="1-16" drill="0.6"/>
-<wire x1="15.494" y1="16.51" x2="15.24" y2="16.764" width="0.254" layer="16"/>
-<wire x1="14.097" y1="16.958" x2="15.046" y2="16.958" width="0.254" layer="16"/>
-<wire x1="15.046" y1="16.958" x2="15.494" y2="16.51" width="0.254" layer="16"/>
-<wire x1="16.394" y1="14.224" x2="16.394" y2="15.61" width="0.254" layer="16"/>
-<wire x1="16.394" y1="15.61" x2="15.494" y2="16.51" width="0.254" layer="16"/>
 <wire x1="14.097" y1="16.958" x2="14.097" y2="18.669" width="0.254" layer="16"/>
 <wire x1="14.097" y1="18.669" x2="13.716" y2="19.05" width="0.254" layer="16"/>
@@
 <wire x1="9.652" y1="19.05" x2="8.382" y2="20.32" width="0.254" layer="16"/>
 <wire x1="8.382" y1="20.32" x2="8.382" y2="23.484" width="0.254" layer="16"/>
+<wire x1="16.394" y1="12.7" x2="16.394" y2="14.224" width="0.254" layer="16"/>
+<wire x1="16.394" y1="14.224" x2="16.394" y2="15.864" width="0.254" layer="16"/>
+<wire x1="16.394" y1="15.864" x2="15.3" y2="16.958" width="0.254" layer="16"/>
+<wire x1="14.097" y1="16.958" x2="15.3" y2="16.958" width="0.254" layer="16"/>
 </signal>
 <signal name="-5V">

Commit message: updated schematic
Parts:
- U$4: value FRAME_SW_LOGO_CC_BY_SA -> FRAME_MINIPH
Changed lines of the file:
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@@
 <layer number="110" name="fp0" color="7" fill="1" visible="no" active="yes"/>
 <layer number="111" name="LPC17xx" color="7" fill="1" visible="yes" active="yes"/>
+<layer number="112" name="tSilk" color="7" fill="1" visible="yes" active="yes"/>
 <layer number="116" name="Patch_BOT" color="9" fill="4" visible="no" active="yes"/>
 <layer number="121" name="_tsilk" color="7" fill="1" visible="no" active="yes"/>
@@
 <layer number="124" name="bTestmark" color="7" fill="1" visible="no" active="yes"/>
 <layer number="125" name="_tNames" color="7" fill="1" visible="no" active="yes"/>
+<layer number="126" name="_bNames" color="7" fill="1" visible="yes" active="yes"/>
+<layer number="127" name="_tValues" color="7" fill="1" visible="yes" active="yes"/>
+<layer number="128" name="_bValues" color="7" fill="1" visible="yes" active="yes"/>
 <layer number="131" name="tAdjust" color="7" fill="1" visible="no" active="yes"/>
 <layer number="132" name="bAdjust" color="7" fill="1" visible="no" active="yes"/>
 <layer number="144" name="Drill_legend" color="7" fill="1" visible="no" active="yes"/>
 <layer number="151" name="HeatSink" color="7" fill="1" visible="no" active="yes"/>
+<layer number="152" name="_bDocu" color="7" fill="1" visible="yes" active="yes"/>
 <layer number="199" name="Contour" color="7" fill="1" visible="yes" active="yes"/>
 <layer number="200" name="200bmp" color="1" fill="10" visible="yes" active="yes"/>
@@
 <layer number="223" name="223bmp" color="24" fill="1" visible="no" active="no"/>
 <layer number="224" name="224bmp" color="25" fill="1" visible="no" active="no"/>
+<layer number="248" name="Housing" color="7" fill="1" visible="yes" active="yes"/>
+<layer number="249" name="Edge" color="7" fill="1" visible="yes" active="yes"/>
 <layer number="250" name="Descript" color="3" fill="1" visible="no" active="no"/>
 <layer number="251" name="SMDround" color="12" fill="11" visible="no" active="no"/>
@@
 <element name="C3" library="SparkysWidgets" package="0805" value=".1uF" x="17.526" y="24.638" rot="MR270"/>
 <element name="SJ1" library="SparkFun" package="SJ_2S-NOTRACE" value="SOLDERJUMPERNC2" x="21.209" y="19.177" smashed="yes" rot="R270"/>
-<element name="U$4" library="SparkysWidgets" package="SWPCBLOGOWITHINFO" value="FRAME_SW_LOGO_CC_BY_SA" x="-22.352" y="-5.334">
-<attribute name="URL1" value="/Projects.aspx" x="-22.352" y="-5.334" size="0.6096" layer="27" display="off"/>
+<element name="U$4" library="SparkysWidgets" package="SWPCBLOGOWITHINFO" value="FRAME_MINIPH" x="-22.352" y="-5.334">
+<attribute name="URL1" value="/portfolio-item/miniph-i2c-ph-interface/" x="-22.352" y="-5.334" size="0.6096" layer="27" display="off"/>
 <attribute name="URLHOME" value="http://www.sparkyswidgets.com" x="-22.352" y="-5.334" size="0.6096" layer="27" display="off"/>
 <attribute name="URLPROJECT" value="http://www.sparkyswidgets.com" x="-22.352" y="-5.334" size="0.6096" layer="27" display="off"/>
-<attribute name="PROJECT" value="I2C ADC Breakout with vRef" x="-22.352" y="-5.334" size="0.6096" layer="27" display="off"/>
+<attribute name="PROJECT" value="Mini pH I2C pH Interface" x="-22.352" y="-5.334" size="0.6096" layer="27" display="off"/>
 </element>
 <element name="U$5" library="SparkysWidgets" package="CC-BY-SA" value="CC-BY-SA" x="-23.114" y="-11.938"/>
