File: MinipHV3_1.brd (EAGLE design)
At the start: 27.9 x 27.9 mm, 33 parts, among them IC1 MCP3221, IC4 TL072, IC5 TPS60400DBV

Commit message: Cleaned up design a bit, added changed to readme
Parts:
- removed SJ1: SOLDERJUMPERNC2, SparkFun:SJ_2S-NOTRACE
- added C5, C7: .1uF, SparkysWidgets:0805
- added C6: 220pF, SparkysWidgets:0805
- added R3: 22, SparkysWidgets:0805
- added T1: (no value), SparkysWidgets:SOT-23
- C1: value 10uF -> 1uF
- IC4: value TL072 -> LMP7702
- JP6: value M01PTH_LONGPAD -> M01PTH; device SparkFun:1X01_LONGPAD -> SparkFun:1X01
- R10, R8, R9: value 220K -> 200K
- R11: value 4.7K -> 500
- R7: value 47K -> 100K
- U$6: value MCP1541 -> REF3030
- moved U$5 25.2 mm to (2.03, -10.9)
- moved U$4 24.1 mm to (1.78, -4.83)
- moved U$1 14.3 mm to (4.32, 6.86), flipped to the bottom
- moved C10 4.60 mm to (2.29, 13.0), turned to 90 degrees
- moved C11 4.50 mm to (3.56, 17.0), turned to 270 degrees
- moved C3 2.69 mm to (18.4, 22.1), turned to 180 degrees
- moved C12 2.29 mm to (8.13, 11.9), turned to 270 degrees
- moved IC5 1.93 mm to (5.08, 13.0)
- moved R11 1.14 mm to (16.5, 25.4), turned to 0 degrees
- moved C2 1.05 mm to (22.4, 20.6)
- moved IC4 0.51 mm to (12.7, 19.6)
- moved JP6 0.36 mm to (19.8, 25.1)
- moved U$6 0.25 mm to (18.5, 19.1)
Connections:
- new net N$4: C11.2, IC5.1, R3.2
- new net VIN: J1.3, JP5.3, T1.1
- net +5V: now also C5.1, T1.2; no longer J1.3, JP5.3, R12.1, SJ1.2
- net -5V: now also C7.2, R3.1; no longer C11.2, IC5.1
- net GND: now also C5.2, C6.2, C7.1, T1.3
- net PHVO: now also C6.1
- net VREF: now also R12.1; no longer SJ1.1
Routing:
- net VIN: track 0.00 -> 30.0 mm
- net VREF: track 8.93 -> 25.5 mm
- net +5V: track 64.7 -> 50.5 mm, vias 1 -> 4
- net N$5: track 34.9 -> 44.2 mm, vias 0 -> 2
- net N$4: track 0.00 -> 4.80 mm
- net N$1: track 9.45 -> 6.69 mm
- net N$2: track 7.80 -> 5.51 mm
- net -5V: track 5.40 -> 4.05 mm
- net N$23: track 2.85 -> 1.51 mm
- net PHVO: track 7.09 -> 8.14 mm
- net N$10: track 17.2 -> 16.6 mm
Other:
- board text added: "Ver 3.0"
- board text removed: "Ver 0.1"
