File: MinipHV3_1.sch (EAGLE design)
At the start: 31 parts, among them IC1 MCP3221, IC4 TL072, IC5 TPS60400DBV

Commit message: Cleaned up design a bit, added changed to readme
Parts:
- removed SJ1: SOLDERJUMPERNC2, SparkFun:SOLDERJUMPERNC2
- added C5, C7: .1uF, SparkysWidgets:CAP0805
- added C6: 220pF, SparkysWidgets:CAP0805
- added R3: 22, SparkysWidgets:RESISTOR0805-RES
- added T1: (no value), SparkysWidgets:PMOSSOT23
- C1: value 10uF -> 1uF
- IC4: value TL072 -> LMP7702
- JP6: value M01PTH_LONGPAD -> M01PTH; device SparkFun:M01PTH_LONGPAD -> SparkFun:M01PTH
- R10, R8, R9: value 220K -> 200K
- R11: value 4.7K -> 500
- R7: value 47K -> 100K
- U$6: value MCP1541 -> REF3030
Connections:
- new net N$4: C11.2, IC5.OUT, R3.2
- new net VIN: J1.3, JP5.3, T1.D
- net +5V: now also C5.1, T1.S; no longer J1.3, JP5.3, R12.1, SJ1.2
- net -5V: now also C7.2, R3.1; no longer C11.2, IC5.OUT
- net GND: now also C5.2, C6.2, C7.1, T1.G
- net PHVO: now also C6.1
- net VREF: now also R12.1; no longer SJ1.1
Other:
- note added: "ADC supplied by stable Vref Using REF3030 (3.0V Vref) VStep = 3.0V/4096Steps = .000732V/step or 732uV per step, .1pH change = 5.916mV 5916uV/732uV = 8.08steps/ .1pH change Vread = Steps/4095 * VREF(3V)"
- note added: "Depenidng on pH probe noise ouput as much as 500uV to 5mV (VPP) (.01pH -.1pH precision over time) RC filter could be added between BNC and Op-amp input but breaks ideal matching to probes impedence (Guard ring hard to implement) DSP LPF @ 7-15Hz works well"
- note added: "G = R8/R7 + 1 = 3"
- note added: "LPF Fc=72.3KHz Fswitch = 250KHz Place C7 near -rail of Op-Amp"
- note added: "Op-Amp power rails Place caps close to pins -rail caps from chargepump"
- note added: "Output Drive and LPF matched to MCP3221 Resoultion, Tacq and CSample 12Bit , 1.12uS , 20pF"
- note added: "PHVout = 1.5V - (-1.242V) = 2.742V PHVout = 1.5V - 1.242 = .258V Range = 2.484V (But of course :)"
- note added: "PHVout= (2*Voffset) - PHgout"
- note added: "PHgol = -.414V*3 =-1.242V PHgoh = .414V*3 = 1.242V Range = 2.484V"
- note added: "Reverse Voltage Protection"
- note added: "Voffset = VREF*R13/(R13+R12)=.750V"
- note added: "Vsupply range = 3.025 - 5.5V"
- moved on the sheet: C1, C10, C11, C12, C2, C3, C9, IC1, IC4A, IC4B, IC5, J1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
